File: build/build7/Interposer/Interposer.kicad_pcb (KiCad board)
At the start: 2 copper layers, 3.6 x 4 mm, 2 parts, among them U1 BQ21040DBVR, U2 BQ21040DBVR

Commit message: Current status: debugged and fixed 4 boards, need to finalize firmware and finish building these 4. All lamps from first build came unglued, need to revise design/assembly to fix this
Connections:
- net Net-(U1-GND) renamed /CHG_N
- net Net-(U1-ISET) renamed /TS
- net Net-(U1-TS) renamed /ISET
- net Net-(U1-VIN) renamed /Vout
- net Net-(U1-~{CHG}) renamed /GND
Changed lines of the file:
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@@
 	)
 	(setup
+		(stackup
+			(layer "F.SilkS"
+				(type "Top Silk Screen")
+			)
+			(layer "F.Paste"
+				(type "Top Solder Paste")
+			)
+			(layer "F.Mask"
+				(type "Top Solder Mask")
+				(thickness 0.01)
+			)
+			(layer "F.Cu"
+				(type "copper")
+				(thickness 0.035)
+			)
+			(layer "dielectric 1"
+				(type "core")
+				(thickness 1.51)
+				(material "FR4")
+				(epsilon_r 4.5)
+				(loss_tangent 0.02)
+			)
+			(layer "B.Cu"
+				(type "copper")
+				(thickness 0.035)
+			)
+			(layer "B.Mask"
+				(type "Bottom Solder Mask")
+				(thickness 0.01)
+			)
+			(layer "B.Paste"
+				(type "Bottom Solder Paste")
+			)
+			(layer "B.SilkS"
+				(type "Bottom Silk Screen")
+			)
+			(copper_finish "None")
+			(dielectric_constraints no)
+		)
 		(pad_to_mask_clearance 0)
 		(allow_soldermask_bridges_in_footprints no)
@@
 	(net 0 "")
 	(net 1 "+5V_USB")
-	(net 2 "Net-(U1-VIN)")
-	(net 3 "Net-(U1-TS)")
-	(net 4 "Net-(U1-GND)")
-	(net 5 "Net-(U1-~{CHG})")
-	(net 6 "Net-(U1-ISET)")
+	(net 2 "/Vout")
+	(net 3 "/ISET")
+	(net 4 "/CHG_N")
+	(net 5 "/GND")
+	(net 6 "/TS")
 	(footprint "salt_booklamp_footprints:BQ21040DBVR"
 		(layer "F.Cu")
@@
 			(layers "F.Cu" "F.Mask" "F.Paste")
 			(roundrect_rratio 0.08333333333)
-			(net 6 "Net-(U1-ISET)")
+			(net 6 "/TS")
 			(pinfunction "TS")
 			(pintype "passive")
@@
 			(layers "F.Cu" "F.Mask" "F.Paste")
 			(roundrect_rratio 0.08333333333)
-			(net 2 "Net-(U1-VIN)")
+			(net 2 "/Vout")
 			(pinfunction "VOUT")
 			(pintype "passive")
@@
 			(layers "F.Cu" "F.Mask" "F.Paste")
 			(roundrect_rratio 0.08333333333)
-			(net 4 "Net-(U1-GND)")
+			(net 4 "/CHG_N")
 			(pinfunction "~{CHG}")
 			(pintype "passive")
@@
 			(layers "F.Cu" "F.Mask" "F.Paste")
 			(roundrect_rratio 0.08333333333)
-			(net 3 "Net-(U1-TS)")
+			(net 3 "/ISET")
 			(pinfunction "ISET")
 			(pintype "passive")
@@
 			(layers "F.Cu" "F.Mask" "F.Paste")
 			(roundrect_rratio 0.08333333333)
-			(net 5 "Net-(U1-~{CHG})")
+			(net 5 "/GND")
 			(pinfunction "GND")
 			(pintype "passive")
@@
 			(layers "B.Cu" "B.Mask" "B.Paste")
 			(roundrect_rratio 0.08333333333)
-			(net 3 "Net-(U1-TS)")
+			(net 3 "/ISET")
 			(pinfunction "TS")
 			(pintype "passive")
@@
 			(layers "B.Cu" "B.Mask" "B.Paste")
 			(roundrect_rratio 0.08333333333)
-			(net 5 "Net-(U1-~{CHG})")
+			(net 5 "/GND")
 			(pinfunction "~{CHG}")
 			(pintype "passive")
@@
 			(layers "B.Cu" "B.Mask" "B.Paste")
 			(roundrect_rratio 0.08333333333)
-			(net 6 "Net-(U1-ISET)")
+			(net 6 "/TS")
 			(pinfunction "ISET")
 			(pintype "passive")
@@
 			(layers "B.Cu" "B.Mask" "B.Paste")
 			(roundrect_rratio 0.08333333333)
-			(net 4 "Net-(U1-GND)")
+			(net 4 "/CHG_N")
 			(pinfunction "GND")
 			(pintype "passive")
@@
 			(layers "B.Cu" "B.Mask" "B.Paste")
 			(roundrect_rratio 0.08333333333)
-			(net 2 "Net-(U1-VIN)")
+			(net 2 "/Vout")
 			(pinfunction "VIN")
 			(pintype "passive")
